File: DplusSim.sch (KiCad schematic (older format))
At the start: 19 parts, among them J10 K15 -, J11 Summer +, J3 Summer -, J7 Landstr. +, J8 Landstr. -, J9 K15 +, Q2 IRF7404, U5 LTV-847

Commit message: x
Parts:
- removed F2: Polyfuse, Resistor_SMD:R_0603_1608Metric_Pad1.05x0.95mm_HandSolder, symbol Device:Polyfuse
- removed H5, H6: MountingHole, MountingHole:MountingHole_2.2mm_M2, symbol Mechanical:MountingHole
- removed J10: K15 -, MyComponents:FASTON-6_3mm, symbol Connector:Conn_01x01_Male
- removed J9: K15 +, MyComponents:FASTON-6_3mm, symbol Connector:Conn_01x01_Male
- added C1: 100n, Capacitor_SMD:C_0805_2012Metric_Pad1.15x1.40mm_HandSolder, symbol Device:C
- added C2, C3, C4: C, Capacitor_SMD:C_0805_2012Metric_Pad1.15x1.40mm_HandSolder, symbol Device:C
- added J1: Conn_02x07_Odd_Even, Connector_PinHeader_1.27mm:PinHeader_2x07_P1.27mm_Vertical, symbol Connector_Generic:Conn_02x07_Odd_Even
- added J2: Conn_01x10, Connector_PinHeader_2.54mm:PinHeader_1x10_P2.54mm_Vertical, symbol Connector_Generic:Conn_01x10
- added J4, J5: Conn_01x08, Connector_PinHeader_2.54mm:PinHeader_1x08_P2.54mm_Vertical, symbol Connector_Generic:Conn_01x08
- added J6: 12V Starter, MyComponents:FASTON-6_3mm, symbol Connector:Conn_01x01_Male
- added R1, R2: R, Resistor_SMD:R_0805_2012Metric_Pad1.15x1.40mm_HandSolder, symbol Device:R
- added U1: LT1117-3.3, Package_TO_SOT_SMD:SOT-223, symbol Regulator_Linear:LT1117-3.3
- added U2: STM32L031F4Px, Package_SO:TSSOP-20_4.4x6.5mm_P0.65mm, symbol MCU_ST_STM32L0:STM32L031F4Px
- J11: value Summer + -> D+
- J3: value Summer - -> GND Starter
- J7: value Landstr. + -> 12V Bord
- J8: value Landstr. - -> GND Bord
Connections:
- net K15_minus is gone; now on net GND: U5.8
- net +12V: now also C3.1, U1.3 (VI); no longer Q2.1 (S), Q2.2 (S), Q2.3 (S), R8.2
- net GND: now also C1.2, C2.2, C3.2, C4.2, J1.11 (Pin_11), J1.5 (Pin_5), J1.7 (Pin_7), J2.2 (Pin_2), R2.2, U1.1 (GND), U2.15 (VSS); no longer J3.1 (Pin_1), U5.9
- net K15_plus renamed Dplus_out
- net Dplus_out: now also U2.9 (PA3)
- net Warn_plus renamed Dplus
- new net: R2.1, U2.1 (BOOT0)
- new net: J4.1 (Pin_1), J5.1 (Pin_1)
- new net: J4.2 (Pin_2), J5.2 (Pin_2)
- new net: J4.3 (Pin_3), J5.3 (Pin_3)
- new net: J4.4 (Pin_4), J5.4 (Pin_4)
- new net: J4.5 (Pin_5), J5.5 (Pin_5)
- new net: J4.6 (Pin_6), J5.6 (Pin_6)
- new net: J4.7 (Pin_7), J5.7 (Pin_7)
- new net: J4.8 (Pin_8), J5.8 (Pin_8)
- new net +12VA: J6.1 (Pin_1), Q2.1 (S), Q2.2 (S), Q2.3 (S), R8.2
- new net +3V3: C1.1, C4.1, J1.3 (Pin_3), J2.1 (Pin_1), R1.2, U1.2 (VO), U2.16 (VDD), U2.5 (VDDA)
- new net EN: J2.6 (Pin_6), U2.7 (PA1)
- new net GNDA: J3.1 (Pin_1), U5.9
- new net I2C_SCL: J2.3 (Pin_3), U2.17 (PA9)
- new net I2C_SDA: J2.4 (Pin_4), U2.18 (PA10)
- new net INT: J2.5 (Pin_5), U2.6 (PA0)
- new net NRST: C2.1, J1.12 (Pin_12), R1.1, U2.4 (NRST)
- new net SPI_MISO: J2.9 (Pin_9), U2.12 (PA6)
- new net SPI_MOSI: J2.10 (Pin_10), U2.13 (PA7)
- new net SPI_NSS: J2.7 (Pin_7), U2.10 (PA4)
- new net SPI_SCK: J2.8 (Pin_8), U2.11 (PA5)
- new net SWDCLK: J1.6 (Pin_6), U2.20 (PA14)
- new net SWDIO: J1.4 (Pin_4), U2.19 (PA13)
- new net USART1_RX: J1.14 (Pin_14)
- new net USART1_TX: J1.13 (Pin_13)
- no-connect marks 0 -> 2
